File: kicad/l6230driver/l6230driver.kicad_sch (KiCad schematic)
At the start: 57 parts, among them J1 Conn_01x02_Female, J2 Conn_01x03_Female, J3 Conn_01x01_Female, J4 Conn_01x02_Female, J5 Conn_01x02_Female, J6 Conn_01x02_Female, J7 Conn_01x04_Female, J8 Conn_01x02_Female, J9 Conn_01x04_Female, U1 L6230PD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

Commit message: added HSOP-36 footprint to own pritty-lib, placing, routing
Parts:
- U1: footprint Package_SO:HSOP-36-1EP_11.0x15.9mm_P0.65mm_SlugDown_ThermalVias -> L6230:HSOP-36
Changed lines of the file:
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@@
     (property "Reference" "U1" (id 0) (at 133.35 40.259 0))
     (property "Value" "L6230PD" (id 1) (at 133.35 42.5704 0))
-    (property "Footprint" "Package_SO:HSOP-36-1EP_11.0x15.9mm_P0.65mm_SlugDown_ThermalVias" (id 2) (at 151.13 90.17 0)
+    (property "Footprint" "L6230:HSOP-36" (id 2) (at 151.13 90.17 0)
       (effects (font (size 1.27 1.27)) hide)
     )
@@
     )
     (path "/00000000-0000-0000-0000-00006317826e"
-      (reference "U1") (unit 1) (value "L6230PD") (footprint "Package_SO:HSOP-36-1EP_11.0x15.9mm_P0.65mm_SlugDown_ThermalVias")
+      (reference "U1") (unit 1) (value "L6230PD") (footprint "L6230:HSOP-36")
     )
     (path "/00000000-0000-0000-0000-0000633d9825"

Commit message: 100% routed
Connections:
- net GND: now also U1.28 (CP-)
- net at R17.2, U3.1: now also J9.2 (Pin_2); no longer J9.1 (Pin_1)
- net at R21.2, U3.7: now also J9.1 (Pin_1); no longer J9.2 (Pin_2)
Other:
- note added: "V U W"
Changed lines of the file:
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@@
   (junction (at 217.17 97.79) (diameter 0) (color 0 0 0 0)
   )
+  (junction (at 113.03 127) (diameter 0) (color 0 0 0 0)
+  )
   (junction (at 158.75 74.93) (diameter 0) (color 0 0 0 0)
   )
@@
   (junction (at 77.47 128.27) (diameter 0) (color 0 0 0 0)
   )
+  (junction (at 49.53 139.7) (diameter 0) (color 0 0 0 0)
+  )
   (junction (at 231.14 85.09) (diameter 0) (color 0 0 0 0)
   )
   (junction (at 77.47 146.05) (diameter 0) (color 0 0 0 0)
   )
-  (junction (at 49.53 139.7) (diameter 0) (color 0 0 0 0)
-  )
   (junction (at 82.55 29.21) (diameter 0) (color 0 0 0 0)
   )
@@
     (stroke (width 0) (type default) (color 0 0 0 0))
   )
-  (wire (pts (xy 38.1 137.16) (xy 44.45 137.16))
-    (stroke (width 0) (type default) (color 0 0 0 0))
-  )
   (wire (pts (xy 95.25 69.85) (xy 69.85 69.85))
     (stroke (width 0) (type default) (color 0 0 0 0))
@@
     (stroke (width 0) (type default) (color 0 0 0 0))
   )
+  (wire (pts (xy 153.67 127) (xy 153.67 85.09))
+    (stroke (width 0) (type default) (color 0 0 0 0))
+  )
   (wire (pts (xy 49.53 157.48) (xy 49.53 163.83))
     (stroke (width 0) (type default) (color 0 0 0 0))
@@
     (stroke (width 0) (type default) (color 0 0 0 0))
   )
+  (wire (pts (xy 49.53 137.16) (xy 49.53 139.7))
+    (stroke (width 0) (type default) (color 0 0 0 0))
+  )
   (wire (pts (xy 236.22 137.16) (xy 231.14 137.16))
     (stroke (width 0) (type default) (color 0 0 0 0))
@@
     (stroke (width 0) (type default) (color 0 0 0 0))
   )
-  (wire (pts (xy 44.45 137.16) (xy 44.45 121.92))
-    (stroke (width 0) (type default) (color 0 0 0 0))
-  )
   (wire (pts (xy 200.66 20.32) (xy 82.55 20.32))
     (stroke (width 0) (type default) (color 0 0 0 0))
@@
     (stroke (width 0) (type default) (color 0 0 0 0))
   )
+  (wire (pts (xy 44.45 121.92) (xy 44.45 139.7))
+    (stroke (width 0) (type default) (color 0 0 0 0))
+  )
   (wire (pts (xy 82.55 20.32) (xy 82.55 29.21))
     (stroke (width 0) (type default) (color 0 0 0 0))
@@
     (stroke (width 0) (type default) (color 0 0 0 0))
   )
-  (wire (pts (xy 113.03 125.73) (xy 113.03 123.19))
+  (wire (pts (xy 113.03 130.81) (xy 113.03 127))
     (stroke (width 0) (type default) (color 0 0 0 0))
   )
@@
     (stroke (width 0) (type default) (color 0 0 0 0))
   )
-  (wire (pts (xy 49.53 139.7) (xy 38.1 139.7))
-    (stroke (width 0) (type default) (color 0 0 0 0))
-  )
   (wire (pts (xy 168.91 72.39) (xy 172.72 72.39))
     (stroke (width 0) (type default) (color 0 0 0 0))
@@
     (stroke (width 0) (type default) (color 0 0 0 0))
   )
+  (wire (pts (xy 153.67 85.09) (xy 151.13 85.09))
+    (stroke (width 0) (type default) (color 0 0 0 0))
+  )
   (wire (pts (xy 151.13 49.53) (xy 177.8 49.53))
     (stroke (width 0) (type default) (color 0 0 0 0))
@@
     (stroke (width 0) (type default) (color 0 0 0 0))
   )
+  (wire (pts (xy 113.03 127) (xy 153.67 127))
+    (stroke (width 0) (type default) (color 0 0 0 0))
+  )
   (wire (pts (xy 254 152.4) (xy 251.46 152.4))
     (stroke (width 0) (type default) (color 0 0 0 0))
@@
     (stroke (width 0) (type default) (color 0 0 0 0))
   )
+  (wire (pts (xy 38.1 139.7) (xy 44.45 139.7))
+    (stroke (width 0) (type default) (color 0 0 0 0))
+  )
+  (wire (pts (xy 113.03 127) (xy 113.03 123.19))
+    (stroke (width 0) (type default) (color 0 0 0 0))
+  )
   (wire (pts (xy 261.62 116.84) (xy 264.16 116.84))
     (stroke (width 0) (type default) (color 0 0 0 0))
@@
     (stroke (width 0) (type default) (color 0 0 0 0))
   )
+  (wire (pts (xy 38.1 137.16) (xy 49.53 137.16))
+    (stroke (width 0) (type default) (color 0 0 0 0))
+  )
   (wire (pts (xy 64.77 124.46) (xy 64.77 128.27))
     (stroke (width 0) (type default) (color 0 0 0 0))
+  )
+  (text "V\nU\nW" (at 27.94 142.24 0)
+    (effects (font (size 1.27 1.27)) (justify left bottom))
   )
   (text "push-pull" (at 66.04 60.96 0)
@@
     (pin "1")
   )
-  (symbol (lib_id "power:GNDPWR") (at 113.03 125.73 0) (unit 1)
-    (in_bom yes) (on_board yes)
-    (property "Reference" "#PWR0106" (id 0) (at 113.03 130.81 0)
-      (effects (font (size 1.27 1.27)) hide)
-    )
-    (property "Value" "GNDPWR" (id 1) (at 113.1316 129.6416 0))
-    (property "Footprint" "" (id 2) (at 113.03 127 0)
-      (effects (font (size 1.27 1.27)) hide)
-    )
-    (property "Datasheet" "" (id 3) (at 113.03 127 0)
-      (effects (font (size 1.27 1.27)) hide)
-    )
+  (symbol (lib_id "power:GNDPWR") (at 113.03 130.81 0) (unit 1)
+    (in_bom yes) (on_board yes)
+    (property "Reference" "#PWR0106" (id 0) (at 113.03 135.89 0)
+      (effects (font (size 1.27 1.27)) hide)
+    )
+    (property "Value" "GNDPWR" (id 1) (at 113.1316 134.7216 0))
+    (property "Footprint" "" (id 2) (at 113.03 132.08 0)
+      (effects (font (size 1.27 1.27)) hide)
+    )
+    (property "Datasheet" "" (id 3) (at 113.03 132.08 0)
+      (effects (font (size 1.27 1.27)) hide)
+    )
